File: audio_codec.kicad_sch (KiCad schematic)
At the start: 22 parts, among them J2 AudioOutput, J3 AudioInput, J4 AudioOutput, U2 WM8731SEDS, U5 TPA6110A2DGN

Commit message: Audio schematic updated
Parts:
- removed RV1: R_Potentiometer_Dual, symbol Device:R_Potentiometer_Dual
- added C?: 470, symbol Device:C
- added C? (x2): 100n, symbol Device:C
- added C?: 470n, symbol Device:C
- added C? (x2): 220p, symbol Device:C
- added C? (x2): 100u, symbol Device:C
- added R? (x2): 33k, symbol Device:R
- added R? (x2): 220k, symbol Device:R
- added R? (x2): 22k, symbol Device:R
- added R? (x2): 1k, symbol Device:R
- added VolumeControlKnob?: ~, Galerna:RK10J12R0A0B, symbol Galerna:RK10J12R0A0B
- J4: value AudioOutput -> Headphones
Connections:
- net +3.3VA: now also U5.6 (VDD), C?.2
- net AUDIO_L_IN: now also R?.1; no longer C18.1
- net AUDIO_L_OUT: now also VolumeControlKnob?.4 (P4)
- net AUDIO_R_IN: now also R?.1; no longer C19.1
- net AUDIO_R_OUT: now also VolumeControlKnob?.5 (P5)
- net GND: now also J4.R2, C?.1, C?.1, C?.2, C?.2, R?.1, R?.1, VolumeControlKnob?.1 (P1)
- net HEADPHONE_OUT_L: now also J4.T, C?.2
- net HEADPHONE_OUT_R: now also J4.R1, C?.2
- net at U5.1 (BYPASS): now also C?.2
- net at U5.4 (IN2-): now also R?.1, R?.2
- net at U5.5 (VO2): now also C?.1, R?.2
- net at U5.7 (VO1): now also C?.1, R?.2
- net at U5.8 (IN1-): now also R?.1, R?.2
- new net: C?.2, R?.1 (x2)
- new net: C18.1, C?.1, R?.2, R?.2
- new net: C19.1, C?.1, R?.2, R?.2
- new net AUDIO_WIPER_OUT_L: C?.1, VolumeControlKnob?.3 (P3)
- new net AUDIO_WIPER_OUT_R: C?.1, VolumeControlKnob?.2 (P2)
- no-connect marks 9 -> 10
Other:
- moved on the sheet: C10, C11, C12, C13, C14, C15, C16, C17, C18, C19, C8, C9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

Commit message: extending library
Parts:
- J2, J3: footprint Connector_Audio:Jack_3.5mm_PJ320D_Horizontal -> Galerna:AUDIO-SMD_PJ-320D-1
- gave numbers to parts that had none: 17
Changed lines of the file:
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@@
 		(dnp no)
 		(fields_autoplaced yes)
-		(property "Reference" "#PWR?"
+		(property "Reference" "#PWR04"
 			(at 234.95 81.28 0)
 			(effects
@@
 		(on_board yes)
 		(dnp no)
-		(property "Reference" "#PWR?"
+		(property "Reference" "#PWR01"
 			(at 233.68 116.84 0)
 			(effects
@@
 		(on_board yes)
 		(dnp no)
-		(property "Reference" "R?"
+		(property "Reference" "R4"
 			(at 214.63 151.13 90)
 			(effects
@@
 		(on_board yes)
 		(dnp no)
-		(property "Reference" "C?"
+		(property "Reference" "C2"
 			(at 177.8 132.588 90)
 			(effects
@@
 		(dnp no)
 		(fields_autoplaced yes)
-		(property "Reference" "R?"
+		(property "Reference" "R6"
 			(at 156.21 22.8599 0)
 			(effects
@@
 		(on_board yes)
 		(dnp no)
-		(property "Reference" "R?"
+		(property "Reference" "R2"
 			(at 187.96 132.08 90)
 			(effects
@@
 		(dnp no)
 		(fields_autoplaced yes)
-		(property "Reference" "#PWR020"
+		(property "Reference" "#PWR?"
 			(at 236.22 41.91 0)
 			(effects
@@
 		(dnp no)
 		(fields_autoplaced yes)
-		(property "Reference" "R6"
+		(property "Reference" "R?"
 			(at 163.83 49.53 90)
 			(effects
@@
 		(dnp no)
 		(fields_autoplaced yes)
-		(property "Reference" "J3"
+		(property "Reference" "J?"
 			(at 257.81 29.8449 0)
 			(effects
@@
 			)
 		)
-		(property "Footprint" "Connector_Audio:Jack_3.5mm_PJ320D_Horizontal"
+		(property "Footprint" "Galerna:AUDIO-SMD_PJ-320D-1"
 			(at 248.92 33.02 0)
 			(effects
@@
 		(dnp no)
 		(fields_autoplaced yes)
-		(property "Reference" "#PWR017"
+		(property "Reference" "#PWR?"
 			(at 105.41 29.21 0)
 			(effects
@@
 		(dnp no)
 		(fields_autoplaced yes)
-		(property "Reference" "#PWR018"
+		(property "Reference" "#PWR?"
 			(at 153.67 95.25 0)
 			(effects
@@
 		(dnp no)
 		(fields_autoplaced yes)
-		(property "Reference" "C17"
+		(property "Reference" "C?"
 			(at 109.22 33.0199 0)
 			(effects
@@
 		(dnp no)
 		(fields_autoplaced yes)
-		(property "Reference" "J2"
+		(property "Reference" "J?"
 			(at 257.81 46.3549 0)
 			(effects
@@
 			)
 		)
-		(property "Footprint" "Connector_Audio:Jack_3.5mm_PJ320D_Horizontal"
+		(property "Footprint" "Galerna:AUDIO-SMD_PJ-320D-1"
 			(at 248.92 49.53 0)
 			(effects
@@
 		(on_board yes)
 		(dnp no)
-		(property "Reference" "#PWR021"
+		(property "Reference" "#PWR?"
 			(at 214.63 152.4 0)
 			(effects
@@
 		(dnp no)
 		(fields_autoplaced yes)
-		(property "Reference" "C14"
+		(property "Reference" "C?"
 			(at 99.06 92.7099 0)
 			(effects
@@
 		(on_board yes)
 		(dnp no)
-		(property "Reference" "#PWR09"
+		(property "Reference" "#PWR?"
 			(at 153.67 73.66 0)
 			(effects
@@
 		(dnp no)
 		(fields_autoplaced yes)
-		(property "Reference" "C?"
+		(property "Reference" "C3"
 			(at 232.41 134.6199 0)
 			(effects
@@
 		(dnp no)
 		(fields_autoplaced yes)
-		(property "Reference" "C?"
+		(property "Reference" "C4"
 			(at 223.52 100.33 90)
 			(effects
@@
 		(dnp no)
 		(fields_autoplaced yes)
-		(property "Reference" "U2"
+		(property "Reference" "U?"
 			(at 73.2633 91.44 0)
 			(effects
@@
 		(dnp no)
 		(fields_autoplaced yes)
-		(property "Reference" "C15"
+		(property "Reference" "C?"
 			(at 113.03 92.7099 0)
 			(effects
@@
 		(dnp no)
 		(fields_autoplaced yes)
-		(property "Reference" "R7"
+		(property "Reference" "R?"
 			(at 156.21 59.6899 0)
 			(effects
@@
 		(dnp no)
 		(fields_autoplaced yes)
-		(property "Reference" "#PWR015"
+		(property "Reference" "#PWR?"
 			(at 30.48 83.82 0)
 			(effects
@@
 		(on_board yes)
 		(dnp no)
-		(property "Reference" "C18"
+		(property "Reference" "C?"
 			(at 147.32 14.986 90)
 			(effects
@@
 		(on_board yes)
 		(dnp no)
-		(property "Reference" "C19"
+		(property "Reference" "C?"
 			(at 147.066 30.226 90)
 			(effects
@@
 		(on_board yes)
 		(dnp no)
-		(property "Reference" "VolumeControlKnob?"
+		(property "Reference" "VolumeControlKnob"
 			(at 134.62 122.682 90)
 			(effects
@@
 		(dnp no)
 		(fields_autoplaced yes)
-		(property "Reference" "C12"
+		(property "Reference" "C?"
 			(at 38.1 33.0199 0)
 			(effects
@@
 		(on_board yes)
 		(dnp no)
-		(property "Reference" "C?"
+		(property "Reference" "C1"
 			(at 177.8 113.792 90)
 			(effects
@@
 		(dnp no)
 		(fields_autoplaced yes)
-		(property "Reference" "#PWR07"
+		(property "Reference" "#PWR?"
 			(at 105.41 53.34 0)
 			(effects
@@
 		(dnp no)
 		(fields_autoplaced yes)
-		(property "Reference" "C9"
+		(property "Reference" "C?"
 			(at 144.78 67.31 90)
 			(effects
@@
 		(dnp no)
 		(fields_autoplaced yes)
-		(property "Reference" "#PWR019"
+		(property "Reference" "#PWR?"
 			(at 236.22 59.69 0)
 			(effects
@@
 		(on_board yes)
 		(dnp no)
-		(property "Reference" "#PWR022"
+		(property "Reference" "#PWR?"
 			(at 151.13 134.62 0)
 			(effects
@@
 		(on_board yes)
 		(dnp no)
-		(property "Reference" "R?"
+		(property "Reference" "R8"
 			(at 171.45 13.716 90)
 			(effects
@@
 		(dnp no)
 		(fields_autoplaced yes)
-		(property "Reference" "C13"
+		(property "Reference" "C?"
 			(at 50.8 33.0199 0)
 			(effects
@@
 		(dnp no)
 		(fields_autoplaced yes)
-		(property "Reference" "R9"
+		(property "Reference" "R?"
 			(at 163.83 68.58 90)
 			(effects
@@
 		(dnp no)
 		(fields_autoplaced yes)
-		(property "Reference" "R?"
+		(property "Reference" "R1"
 			(at 187.96 114.3 90)
 			(effects
@@
 		(on_board yes)
 		(dnp no)
-		(property "Reference" "C8"
+		(property "Reference" "C?"
 			(at 144.78 47.752 90)
 			(effects
@@
 		(dnp no)
 		(fields_autoplaced yes)
-		(property "Reference" "#PWR016"
+		(property "Reference" "#PWR?"
 			(at 109.22 111.76 0)
 			(effects
@@
 		(dnp no)
 		(fields_autoplaced yes)
-		(property "Reference" "J4"
+		(property "Reference" "J?"
 			(at 256.54 69.2149 0)
 			(effects
@@
 		(dnp no)
 		(fields_autoplaced yes)
-		(property "Reference" "R?"
+		(property "Reference" "R3"
 			(at 213.36 86.36 90)
 			(effects
@@
 		(dnp no)
 		(fields_autoplaced yes)
-		(property "Reference" "#PWR?"
+		(property "Reference" "#PWR03"
 			(at 228.6 148.59 0)
 			(effects
@@
 		(dnp no)
 		(fields_autoplaced yes)
-		(property "Reference" "R8"
+		(property "Reference" "R?"
 			(at 156.21 80.0099 0)
 			(effects
@@
 		(on_board yes)
 		(dnp no)
-		(property "Reference" "#PWR01"
+		(property "Reference" "#PWR?"
 			(at 63.5 106.68 0)
 			(effects
@@
 		(dnp no)
 		(fields_autoplaced yes)
-		(property "Reference" "#PWR014"
+		(property "Reference" "#PWR?"
 			(at 21.59 52.07 0)
 			(effects
@@
 		(dnp no)
 		(fields_autoplaced yes)
-		(property "Reference" "C10"
+		(property "Reference" "C?"
 			(at 83.82 33.0199 0)
 			(effects
@@
 		(on_board yes)
 		(dnp no)
-		(property "Reference" "#PWR?"
+		(property "Reference" "#PWR05"
 			(at 153.67 52.07 0)
 			(effects
@@
 		(dnp no)
 		(fields_autoplaced yes)
-		(property "Reference" "C?"
+		(property "Reference" "C8"
 			(at 167.64 36.8299 0)
 			(effects
@@
 		(on_board yes)
 		(dnp no)
-		(property "Reference" "#PWR?"
+		(property "Reference" "#PWR06"
 			(at 153.67 36.83 0)
 			(effects
@@
 		(dnp no)
 		(fields_autoplaced yes)
-		(property "Reference" "#PWR?"
+		(property "Reference" "#PWR02"
 			(at 214.63 106.68 0)
 			(effects
@@
 		(on_board yes)
 		(dnp no)
-		(property "Reference" "C?"
+		(property "Reference" "C5"
 			(at 247.65 116.84 90)
 			(effects
@@
 		(dnp no)
 		(fields_autoplaced yes)
-		(property "Reference" "C11"
+		(property "Reference" "C?"
 			(at 25.4 33.0199 0)
 			(effects
@@
 		(dnp no)
 		(fields_autoplaced yes)
-		(property "Reference" "R?"
+		(property "Reference" "R5"
 			(at 156.21 36.8299 0)
 			(effects
@@
 		(on_board yes)
 		(dnp no)
-		(property "Reference" "C?"
+		(property "Reference" "C6"
 			(at 247.65 129.794 90)
 			(effects
@@
 		(dnp no)
 		(fields_autoplaced yes)
-		(property "Reference" "C16"
+		(property "Reference" "C?"
 			(at 96.52 33.0199 0)
 			(effects
@@
 		(dnp no)
 		(fields_autoplaced yes)
-		(property "Reference" "#PWR013"
+		(property "Reference" "#PWR?"
 			(at 21.59 29.21 0)
 			(effects
@@
 		(dnp no)
 		(fields_autoplaced yes)
-		(property "Reference" "C?"
+		(property "Reference" "C7"
 			(at 167.64 22.8599 0)
 			(effects
@@
 		(on_board yes)
 		(dnp no)
-		(property "Reference" "R?"
+		(property "Reference" "R9"
 			(at 171.45 28.956 90)
 			(effects
@@
 		(dnp no)
 		(fields_autoplaced yes)
-		(property "Reference" "U5"
+		(property "Reference" "U?"
 			(at 216.7733 110.49 0)
 			(effects
