File: audio_codec.kicad_sch (KiCad schematic)
At the start: 38 parts, among them J2 AudioOutput, J3 AudioInput, J4 Headphones, U2 WM8731SEDS, U5 TPA6110A2DGN

Commit message: ERC fixed
Parts:
- U5: footprint 2 -> Package_SO:HVSSOP-8-1EP_3x3mm_P0.65mm_EP1.57x1.89mm
Connections:
- net +3.3VA renamed +3V3A
- net IS2_MCk renamed I2S_MCK
Changed lines of the file:
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@@
 	)
 	(junction
+		(at 63.5 99.06)
+		(diameter 0)
+		(color 0 0 0 0)
+	)
+	(junction
 		(at 92.71 30.48)
 		(diameter 0)
@@
 	(wire
 		(pts
-			(xy 63.5 96.52) (xy 63.5 100.33)
+			(xy 63.5 96.52) (xy 63.5 99.06)
 		)
 		(stroke
@@
 	(wire
 		(pts
+			(xy 63.5 99.06) (xy 63.5 100.33)
+		)
+		(stroke
+			(width 0)
+			(type default)
+		)
+	)
+	(wire
+		(pts
 			(xy 191.77 125.73) (xy 201.93 125.73)
 		)
@@
 		)
 	)
-	(global_label "IS2_MCk"
+	(global_label "I2S_MCK"
 		(shape input)
 		(at 45.72 81.28 180)
@@
 		)
 		(property "Intersheetrefs" "${INTERSHEET_REFS}"
-			(at 34.9939 81.28 0)
+			(at 34.752 81.28 0)
 			(effects
 				(font
@@
 			)
 		)
-		(property "Value" "+3.3VA"
+		(property "Value" "+3V3A"
 			(at 105.41 20.32 0)
 			(effects
@@
 	)
 	(symbol
+		(lib_id "power:PWR_FLAG")
+		(at 63.5 99.06 90)
+		(unit 1)
+		(exclude_from_sim no)
+		(in_bom yes)
+		(on_board yes)
+		(dnp no)
+		(fields_autoplaced yes)
+		(property "Reference" "#FLG04"
+			(at 61.595 99.06 0)
+			(effects
+				(font
+					(size 1.27 1.27)
+				)
+				(hide yes)
+			)
+		)
+		(property "Value" "PWR_FLAG"
+			(at 59.69 99.0599 90)
+			(effects
+				(font
+					(size 1.27 1.27)
+				)
+				(justify left)
+			)
+		)
+		(property "Footprint" ""
+			(at 63.5 99.06 0)
+			(effects
+				(font
+					(size 1.27 1.27)
+				)
+				(hide yes)
+			)
+		)
+		(property "Datasheet" "~"
+			(at 63.5 99.06 0)
+			(effects
+				(font
+					(size 1.27 1.27)
+				)
+				(hide yes)
+			)
+		)
+		(property "Description" "Special symbol for telling ERC where power comes from"
+			(at 63.5 99.06 0)
+			(effects
+				(font
+					(size 1.27 1.27)
+				)
+				(hide yes)
+			)
+		)
+		(pin "1"
+		)
+		(instances
+			(project ""
+				(path "/a77f8f1b-3e6d-40f9-a36e-54a20299e9bc/c8eca522-3096-4cb1-b457-c66eaba9f73c"
+					(reference "#FLG04")
+					(unit 1)
+				)
+			)
+		)
+	)
+	(symbol
 		(lib_id "Galerna:RK10J12R0A0B")
 		(at 134.62 128.27 90)
@@
 			)
 		)
-		(property "Value" "+3.3VA"
+		(property "Value" "+3V3A"
 			(at 212.09 102.87 0)
 			(effects
@@
 			)
 		)
-		(property "Footprint" "2"
+		(property "Footprint" "Package_SO:HVSSOP-8-1EP_3x3mm_P0.65mm_EP1.57x1.89mm"
 			(at 212.09 130.81 0)
 			(effects

Commit message: footprints updated
Parts:
- C200: renamed from C11; footprint (none) -> Capacitor_SMD:C_0603_1608Metric
- C201: renamed from C12; footprint (none) -> Capacitor_SMD:C_0402_1005Metric
- C202: renamed from C13; footprint (none) -> Capacitor_SMD:C_0402_1005Metric
- C203: renamed from C10; footprint (none) -> Capacitor_SMD:C_0402_1005Metric
- C204: renamed from C44; footprint (none) -> Capacitor_SMD:C_0402_1005Metric
- C205: renamed from C45; value 470 -> 470n; footprint (none) -> Capacitor_SMD:C_0402_1005Metric
- C206: renamed from C16; footprint (none) -> Capacitor_SMD:C_0402_1005Metric
- C207: renamed from C14; footprint (none) -> Capacitor_SMD:C_0402_1005Metric
- C208: renamed from C17; footprint (none) -> Capacitor_SMD:C_0603_1608Metric
- C209: renamed from C15; footprint (none) -> Capacitor_SMD:C_0603_1608Metric
- C210: renamed from C46; footprint (none) -> Capacitor_SMD:C_0402_1005Metric
- C211: renamed from C47; footprint (none) -> Capacitor_SMD:C_0402_1005Metric
- C212: renamed from C48; footprint (none) -> Capacitor_SMD:C_0603_1608Metric
- C213: renamed from C49; footprint (none) -> Capacitor_SMD:C_0603_1608Metric
- C214: renamed from C8; footprint (none) -> Capacitor_SMD:C_0805_2012Metric
- C215: renamed from C9; footprint (none) -> Capacitor_SMD:C_0805_2012Metric
- C216: renamed from C18; footprint (none) -> Capacitor_SMD:C_0805_2012Metric
- C217: renamed from C19; footprint (none) -> Capacitor_SMD:C_0805_2012Metric
- C218: renamed from C42; footprint (none) -> Capacitor_SMD:C_0402_1005Metric
- C219: renamed from C43; footprint (none) -> Capacitor_SMD:C_0402_1005Metric
- R200: renamed from R28; footprint (none) -> Resistor_SMD:R_0402_1005Metric
- R201: renamed from R29; footprint (none) -> Resistor_SMD:R_0402_1005Metric
- R202: renamed from R30; footprint (none) -> Resistor_SMD:R_0402_1005Metric
- R203: renamed from R31; footprint (none) -> Resistor_SMD:R_0402_1005Metric
- R204: renamed from R24; footprint (none) -> Resistor_SMD:R_0402_1005Metric
- R205: renamed from R25; footprint (none) -> Resistor_SMD:R_0402_1005Metric
- R206: renamed from R7; footprint (none) -> Resistor_SMD:R_0402_1005Metric
- R207: renamed from R8; footprint (none) -> Resistor_SMD:R_0402_1005Metric
- R208: renamed from R6; footprint (none) -> Resistor_SMD:R_0402_1005Metric
- R209: renamed from R9; footprint (none) -> Resistor_SMD:R_0402_1005Metric
- R210: renamed from R26; footprint (none) -> Resistor_SMD:R_0402_1005Metric
- R211: renamed from R27; footprint (none) -> Resistor_SMD:R_0402_1005Metric
- renumbered J4 to J200, J3 to J201, J2 to J202, U2 to U200, U5 to U201, VolumeControlKnob1 to VolumeControlKnob200
Other:
- note added: "AUDIO CODEC"
- note added: "AUDIO INPUT/OUTPUT"
- note added: "AUDIO INTERFACE"
- note added: "HEADPHONE AMPLIFIER"
- note added: "[2]AUDIO"
- moved on the sheet: C200, C201, C202, C203, C204, C205, C206, C207, C208, C209, C210, C211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
