File: audio_codec.kicad_sch (KiCad schematic)
At the start: 43 parts, among them J2 HEADPHONES, J3 AUDIO_IN, J4 AUDIO_OUT, U2 ES8388, U3 TPA6110A2DGN

Commit message: fillin info in parts
Parts:
- R14, R15: footprint (none) -> Resistor_SMD:R_0402_1005Metric
- R16: LCSC Part (none) -> C470487; Manufacturer (none) -> ALPSALPINE; Manufacturer Part (none) -> RK09L12D0A1W
- U2: LCSC Part (none) -> C365736; Manufacturer (none) -> Everest-semi(Everest Semiconductor); Manufacturer Part (none) -> ES8388
- U3: LCSC Part (none) -> C130212; Manufacturer (none) -> Texas Instruments; Manufacturer Part (none) -> TPA6110A2DGNR

Commit message: JLC order
Parts:
- C21, C26: footprint Capacitor_SMD:C_0603_1608Metric -> Capacitor_SMD:C_0402_1005Metric
- C29, C30: value 470n -> 1u
- R21, R22: value 220k -> 200k
- R27, R28: LCSC Part (none) -> C11702; Manufacturer (none) -> UNI-ROYAL(Uniroyal Elec); Manufacturer Part (none) -> 0402WGF1001TCE
Changed lines of the file:
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@@
 		)
 	)
+	(text_box "C29/30 1u\nR17/18 22k \n\nfc -> 7Hz "
+		(exclude_from_sim no)
+		(at 91.44 185.42 0)
+		(size 26.67 10.16)
+		(margins 0.9525 0.9525 0.9525 0.9525)
+		(stroke
+			(width 0)
+			(type solid)
+		)
+		(fill
+			(type none)
+		)
+		(effects
+			(font
+				(size 1.27 1.27)
+			)
+			(justify left top)
+		)
+	)
 	(text_box "Audio Codec\n===========\n\nDecoupling capacitors\n\nFor each supply pin (or each supply \"domain\" pin):\n\n1× 100 nF MLCC placed right at that pin (same side, shortest loop to GND)\n\nPer rail (shared):\n\n1× bulk cap (typically 4.7-10 µF) near the codec on that rail\n\nThis gives:\n\nHF stability (100 nF)\n\nMF/LF charge storage (bulk)"
 		(exclude_from_sim no)
@@
 			)
 		)
-		(property "Value" "470n"
+		(property "Value" "1u"
 			(at 118.11 221.234 90)
 			(effects
@@
 			)
 		)
-		(property "Value" "220k"
+		(property "Value" "200k"
 			(at 205.74 66.0399 0)
 			(effects
@@
 			)
 		)
-		(property "Footprint" "Capacitor_SMD:C_0603_1608Metric"
+		(property "Footprint" "Capacitor_SMD:C_0402_1005Metric"
 			(at 82.2452 120.65 0)
 			(effects
@@
 			)
 		)
-		(property "Footprint" "Capacitor_SMD:C_0603_1608Metric"
+		(property "Footprint" "Capacitor_SMD:C_0402_1005Metric"
 			(at 46.6852 120.65 0)
 			(effects
@@
 			)
 		)
-		(property "Value" "470n"
+		(property "Value" "1u"
 			(at 118.11 208.026 90)
 			(effects
@@
 			)
 		)
-		(property "Manufacturer Part" ""
+		(property "Manufacturer Part" "0402WGF1001TCE"
+			(at 220.98 59.69 90)
+			(effects
+				(font
+					(size 1.27 1.27)
+				)
+				(hide yes)
+			)
+		)
+		(property "LCSC Part" "C11702"
+			(at 220.98 59.69 90)
+			(effects
+				(font
+					(size 1.27 1.27)
+				)
+				(hide yes)
+			)
+		)
+		(property "Manufacturer" "UNI-ROYAL(Uniroyal Elec)"
 			(at 220.98 59.69 90)
 			(effects
@@
 			)
 		)
-		(property "Value" "220k"
+		(property "Value" "200k"
 			(at 205.74 80.0099 0)
 			(effects
@@
 			)
 		)
-		(property "Manufacturer Part" ""
+		(property "Manufacturer Part" "0402WGF1001TCE"
+			(at 220.98 74.93 90)
+			(effects
+				(font
+					(size 1.27 1.27)
+				)
+				(hide yes)
+			)
+		)
+		(property "LCSC Part" "C11702"
+			(at 220.98 74.93 90)
+			(effects
+				(font
+					(size 1.27 1.27)
+				)
+				(hide yes)
+			)
+		)
+		(property "Manufacturer" "UNI-ROYAL(Uniroyal Elec)"
 			(at 220.98 74.93 90)
 			(effects
