File: input_control.kicad_sch (KiCad schematic)
At the start: 17 parts, among them SW1 100SP1T1B4M2QE, SW2 100SP1T1B4M2QE, U7 CD4051BM

Commit message: fillin info in parts
Parts:
- BTN1, BTN2: MANUFACTURER TE CONNECTIVITY -> (none); Manufacturer (none) -> TE CONNECTIVITY; STANDARD Manufacturer Recommendations -> (none)
- POT_1, POT_2, POT_3, POT_4, POT_5, POT_6, POT_7, POT_8: LCSC Part (none) -> C5848796; Manufacturer (none) -> BOURNS; Manufacturer Part (none) -> PTV09A-4225F-B104
- R34: value 1K -> 1k
- SW1, SW2: LCSC Part (none) -> C273353; MANUFACTURER E-Switch -> (none); Manufacturer (none) -> E-Switch; Manufacturer Part (none) -> 100SP1T1B4M2QE; STANDARD Manufacturer Recommendations -> (none)
- U7: LCSC Part (none) -> C21379; Manufacturer (none) -> Texas Instruments; Manufacturer Part (none) -> CD4051BM96

Commit message: JLC order
Parts:
- R34: LCSC Part (none) -> C11702; Manufacturer (none) -> UNI-ROYAL(Uniroyal Elec); Manufacturer Part (none) -> 0402WGF1001TCE
Changed lines of the file:
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@@
 			)
 		)
-		(property "Manufacturer Part" ""
+		(property "Manufacturer Part" "0402WGF1001TCE"
 			(at 115.57 34.29 90)
 			(effects
+				(font
+					(size 1.27 1.27)
+				)
+				(hide yes)
+			)
+		)
+		(property "LCSC Part" "C11702"
+			(at 115.57 34.29 90)
+			(effects
+				(font
+					(size 1.27 1.27)
+				)
+				(hide yes)
+			)
+		)
+		(property "Manufacturer" "UNI-ROYAL(Uniroyal Elec)"
+			(at 115.57 34.29 90)
+			(effects
