File: mcu.kicad_sch (KiCad schematic)
At the start: 46 parts, among them CN100 HX JN1.27-2X5 TP H4.9, J100 DM3CS-SF, U100 SW_RUN, U101 STM32F405RGTx, X100 X1E000210127000G

Commit message: last status
Connections:
- net PUSH_BTN_0: now also U101.9 (PC1); no longer U101.56 (PB4)
- net PUSH_BTN_1: now also U101.8 (PC0); no longer U101.57 (PB5)
- net SW_0: now also U101.56 (PB4); no longer U101.9 (PC1)
- net SW_1: now also U101.57 (PB5); no longer U101.8 (PC0)
Changed lines of the file:
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@@
 		)
 	)
-	(global_label "SW_1"
+	(global_label "PUSH_BTN_1"
 		(shape input)
 		(at 187.96 76.2 180)
@@
 		)
 		(property "Intersheetrefs" "${INTERSHEET_REFS}"
-			(at 180.1368 76.2 0)
+			(at 173.1215 76.2 0)
 			(effects
 				(font
@@
 		)
 	)
-	(global_label "PUSH_BTN_0"
+	(global_label "SW_0"
 		(shape input)
 		(at 241.3 106.68 0)
@@
 		)
 		(property "Intersheetrefs" "${INTERSHEET_REFS}"
-			(at 256.1385 106.68 0)
+			(at 249.1232 106.68 0)
 			(effects
 				(font
@@
 		)
 	)
-	(global_label "PUSH_BTN_1"
+	(global_label "SW_1"
 		(shape input)
 		(at 241.3 109.22 0)
@@
 		)
 		(property "Intersheetrefs" "${INTERSHEET_REFS}"
-			(at 256.1385 109.22 0)
+			(at 249.1232 109.22 0)
 			(effects
 				(font
@@
 		)
 	)
-	(global_label "SW_0"
+	(global_label "PUSH_BTN_0"
 		(shape input)
 		(at 187.96 78.74 180)
@@
 		)
 		(property "Intersheetrefs" "${INTERSHEET_REFS}"
-			(at 180.1368 78.74 0)
-			(effects
-				(font
+			(at 173.1215 78.74 0)
+			(effects
+				(font

Commit message: Codec updated to ES8388 on schematic
Parts:
- CN1: renamed from CN100; LCSC (none) -> C42372555; LCSC Part C42372555 -> (none)
- J1: renamed from J100; LCSC (none) -> C202111
- SW_1: renamed from U100; value SW_RUN -> BOOT_MODE
- U1: renamed from U101; LCSC (none) -> C15742
- renumbered C100 to C1, C109 to C10, C110 to C11, C111 to C12, C112 to C13, C113 to C14, C114 to C15, C115 to C16, C116 to C17, C117 to C18, C118 to C19, C101 to C2, C102 to C3, C103 to C4, C104 to C5, C105 to C6, C106 to C7, C107 to C8, C108 to C9, D100 to D1, D104 to D2, D101 to D3, D102 to D4, D103 to D5, ER-OLEDM015-2W100 to ER-OLEDM015-2W1, FB100 to FB1, L100 to L1, R100 to R1, R109 to R10, R110 to R11, R111 to R12, R112 to R13, R101 to R2, R102 to R3, R103 to R4, R104 to R5, R105 to R6, R106 to R7, R107 to R8, R108 to R9, SW_100 to SW_2, X100 to X1
Connections:
- net SW_0 renamed SW_2
- net SW_1 renamed SW_3

Commit message: fillin info in parts
Parts:
- CN1: LCSC C42372555 -> (none); LCSC Part (none) -> C42372555; Manufacturer (none) -> HANXIA; Manufacturer Part (none) -> HX JN1.27-2x5 TP H4.9
- D2: Manufacturer (none) -> Born; Manufacturer Part (none) -> RCLAMP0521P-N
- J1: LCSC C202111 -> (none); LCSC Part (none) -> C202111; MANUFACTURER Hirose -> (none); Manufacturer (none) -> Hirose; Manufacturer Part (none) -> DM3CS-SF; STANDARED manufacturer recommendation -> (none)
- R1: value 1K -> 1k
- R3: value 10K -> 10k
- SW_1: Manufacturer (none) -> SHOU HAN; Manufacturer Part (none) -> SS12D10G5
- SW_2: Manufacturer (none) -> XUNPU; Manufacturer Part (none) -> TS-1088-AR02016
- U1: LCSC C15742 -> (none); LCSC Part (none) -> C15742; Manufacturer (none) -> STMicroelectronics; Manufacturer Part (none) -> STM32F405RGT6
- X1: Manufacturer (none) -> Seiko Epson; Manufacturer Part (none) -> X1E0000210127

Commit message: JLC order
Parts:
- removed L1: 10n, Inductor_SMD:L_0402_1005Metric, symbol Device:L
- added FB3: 120@100Mhz, Resistor_SMD:R_0603_1608Metric, symbol Device:FerriteBead
- D1: footprint LED_SMD:LED_0402_1005Metric -> LED_SMD:LED_0603_1608Metric
- D3, D4, D5: value BLUE LED -> YELLOW_LED; footprint LED_SMD:LED_0402_1005Metric -> LED_SMD:LED_0603_1608Metric
- R1: LCSC Part (none) -> C11702; Manufacturer (none) -> UNI-ROYAL(Uniroyal Elec); Manufacturer Part (none) -> 0402WGF1001TCE
- R11, R12, R13: value 330 -> 1k
Connections:
- net +3V3: now also FB3.2
- net VDDA: now also FB3.1
Changed lines of the file:
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@@
 		(on_board yes)
 		(dnp no)
-		(fields_autoplaced yes)
 		(property "Reference" "R12"
-			(at 345.44 104.14 90)
+			(at 345.186 107.696 90)
 			(effects
 				(font
@@
 			)
 		)
-		(property "Value" "330"
-			(at 345.44 106.68 90)
+		(property "Value" "1k"
+			(at 345.44 113.538 90)
 			(effects
 				(font
@@
 			)
 		)
-		(property "Value" "BLUE LED"
+		(property "Value" "YELLOW_LED"
 			(at 356.616 106.68 0)
 			(effects
@@
 			)
 		)
-		(property "Footprint" "LED_SMD:LED_0402_1005Metric"
+		(property "Footprint" "LED_SMD:LED_0603_1608Metric"
 			(at 355.6 110.49 0)
 			(effects
@@
 			)
 		)
-		(property "Footprint" "LED_SMD:LED_0402_1005Metric"
+		(property "Footprint" "LED_SMD:LED_0603_1608Metric"
 			(at 60.96 54.61 0)
 			(effects
@@
 		(on_board yes)
 		(dnp no)
-		(fields_autoplaced yes)
 		(property "Reference" "R11"
-			(at 345.44 90.17 90)
+			(at 345.44 93.472 90)
 			(effects
 				(font
@@
 			)
 		)
-		(property "Value" "330"
-			(at 345.44 92.71 90)
+		(property "Value" "1k"
+			(at 345.694 99.568 90)
 			(effects
 				(font
@@
 	)
 	(symbol
-		(lib_id "Device:L")
-		(at 273.05 31.75 90)
-		(unit 1)
-		(exclude_from_sim no)
-		(in_bom yes)
-		(on_board yes)
-		(dnp no)
-		(fields_autoplaced yes)
-		(property "Reference" "L1"
-			(at 273.05 26.67 90)
-			(effects
-				(font
-					(size 1.27 1.27)
-				)
-			)
-		)
-		(property "Value" "10n"
-			(at 273.05 29.21 90)
-			(effects
-				(font
-					(size 1.27 1.27)
-				)
-			)
-		)
-		(property "Footprint" "Inductor_SMD:L_0402_1005Metric"
-			(at 273.05 31.75 0)
-			(effects
-				(font
-					(size 1.27 1.27)
-				)
-				(hide yes)
-			)
-		)
-		(property "Datasheet" "~"
-			(at 273.05 31.75 0)
-			(effects
-				(font
-					(size 1.27 1.27)
-				)
-				(hide yes)
-			)
-		)
-		(property "Description" "Inductor"
-			(at 273.05 31.75 0)
-			(effects
-				(font
-					(size 1.27 1.27)
-				)
-				(hide yes)
-			)
-		)
-		(property "Manufacturer Part" ""
-			(at 273.05 31.75 90)
-			(effects
-				(font
-					(size 1.27 1.27)
-				)
-				(hide yes)
-			)
-		)
-		(pin "2"
-		)
-		(pin "1"
-		)
-		(instances
-			(project "mcu"
-				(path "/8875c119-10ac-4d8a-bc06-d27618c176ec"
-					(reference "L?")
-					(unit 1)
-				)
-			)
-			(project ""
-				(path "/a77f8f1b-3e6d-40f9-a36e-54a20299e9bc/6f30b934-5b55-48c2-913b-4ebe4ce514c8"
-					(reference "L1")
-					(unit 1)
-				)
-			)
-		)
-	)
-	(symbol
 		(lib_id "MCU_ST_STM32F4:STM32F405RGTx")
 		(at 214.63 93.98 0)
@@
 			)
 		)
-		(property "Value" "BLUE LED"
+		(property "Value" "YELLOW_LED"
 			(at 357.1875 91.44 0)
 			(effects
@@
 			)
 		)
-		(property "Footprint" "LED_SMD:LED_0402_1005Metric"
+		(property "Footprint" "LED_SMD:LED_0603_1608Metric"
 			(at 355.6 96.52 0)
 			(effects
@@
 			)
 		)
-		(property "Value" "BLUE LED"
+		(property "Value" "YELLOW_LED"
 			(at 357.632 123.19 0)
 			(effects
@@
 			)
 		)
-		(property "Footprint" "LED_SMD:LED_0402_1005Metric"
+		(property "Footprint" "LED_SMD:LED_0603_1608Metric"
 			(at 355.6 127 0)
 			(effects
@@
 			)
 		)
-		(property "Manufacturer Part" ""
+		(property "Manufacturer Part" "0402WGF1001TCE"
+			(at 60.96 62.23 0)
+			(effects
+				(font
+					(size 1.27 1.27)
+				)
+				(hide yes)
+			)
+		)
+		(property "LCSC Part" "C11702"
+			(at 60.96 62.23 0)
+			(effects
+				(font
+					(size 1.27 1.27)
+				)
+				(hide yes)
+			)
+		)
+		(property "Manufacturer" "UNI-ROYAL(Uniroyal Elec)"
 			(at 60.96 62.23 0)
 			(effects
@@
 		(on_board yes)
 		(dnp no)
-		(fields_autoplaced yes)
 		(property "Reference" "R13"
-			(at 345.44 120.65 90)
+			(at 345.186 124.46 90)
 			(effects
 				(font
@@
 			)
 		)
-		(property "Value" "330"
-			(at 345.44 123.19 90)
+		(property "Value" "1k"
+			(at 345.694 130.048 90)
 			(effects
 				(font
@@
 					(unit 1)
 				)
+			)
+		)
+	)
+	(symbol
+		(lib_id "Device:FerriteBead")
+		(at 273.05 31.75 90)
+		(unit 1)
+		(exclude_from_sim no)
+		(in_bom yes)
+		(on_board yes)
+		(dnp no)
+		(fields_autoplaced yes)
+		(property "Reference" "FB3"
+			(at 272.9992 24.13 90)
+			(effects
+				(font
+					(size 1.27 1.27)
+				)
+			)
+		)
+		(property "Value" "120@100Mhz"
+			(at 272.9992 26.67 90)
+			(effects
+				(font
+					(size 1.27 1.27)
+				)
+			)
+		)
+		(property "Footprint" "Resistor_SMD:R_0603_1608Metric"
+			(at 273.05 33.528 90)
+			(effects
+				(font
+					(size 1.27 1.27)
+				)
+				(hide yes)
+			)
+		)
+		(property "Datasheet" "~"
+			(at 273.05 31.75 0)
+			(effects
+				(font
+					(size 1.27 1.27)
+				)
+				(hide yes)
+			)
+		)
+		(property "Description" "Ferrite bead"
+			(at 273.05 31.75 0)
+			(effects
+				(font
+					(size 1.27 1.27)
+				)
+				(hide yes)
+			)
+		)
+		(pin "1"
+		)
+		(pin "2"
+		)
+		(instances
+			(project ""
+				(path "/a77f8f1b-3e6d-40f9-a36e-54a20299e9bc/6f30b934-5b55-48c2-913b-4ebe4ce514c8"
+					(reference "FB3")
+					(unit 1)
+				)
